Commit message: TEMP

File: jaguar/arm/install/jaguar_full/share/jaguar_full/config/jaguar_robot_full.ros2_control.xacro (robot description, xacro)
@@ -1,54 +1 @@
-<?xml version="1.0"?>
-<robot xmlns:xacro="http://www.ros.org/wiki/xacro">
-    <xacro:macro name="jaguar_robot_full_ros2_control" params="name initial_positions_file">
-        <xacro:property name="initial_positions" value="${load_yaml(initial_positions_file)['initial_positions']}"/>
-        <ros2_control name="${name}" type="system">
-            <hardware>
-                <!-- By default, set up controllers for simulation. This won't work on real hardware -->
-                <plugin>mock_components/GenericSystem</plugin>
-            </hardware>
-            <joint name="Joint1">
-                <command_interface name="position"/>
-                <state_interface name="position">
-                  <param name="initial_value">${initial_positions['Joint1']}</param>
-                </state_interface>
-                <state_interface name="velocity"/>
-            </joint>
-            <joint name="Joint2">
-                <command_interface name="position"/>
-                <state_interface name="position">
-                  <param name="initial_value">${initial_positions['Joint2']}</param>
-                </state_interface>
-                <state_interface name="velocity"/>
-            </joint>
-            <joint name="Joint3">
-                <command_interface name="position"/>
-                <state_interface name="position">
-                  <param name="initial_value">${initial_positions['Joint3']}</param>
-                </state_interface>
-                <state_interface name="velocity"/>
-            </joint>
-            <joint name="Joint4">
-                <command_interface name="position"/>
-                <state_interface name="position">
-                  <param name="initial_value">${initial_positions['Joint4']}</param>
-                </state_interface>
-                <state_interface name="velocity"/>
-            </joint>
-            <joint name="Joint5">
-                <command_interface name="position"/>
-                <state_interface name="position">
-                  <param name="initial_value">${initial_positions['Joint5']}</param>
-                </state_interface>
-                <state_interface name="velocity"/>
-            </joint>
-            <joint name="Joint6">
-                <command_interface name="position"/>
-                <state_interface name="position">
-                  <param name="initial_value">${initial_positions['Joint6']}</param>
-                </state_interface>
-                <state_interface name="velocity"/>
-            </joint>
-        </ros2_control>
-    </xacro:macro>
-</robot>
+/home/arepo/TMR2026_Rescue/jaguar/arm/src/jaguar_full/config/jaguar_robot_full.ros2_control.xacro

File: jaguar/arm/install/jaguar_full/share/jaguar_full/config/jaguar_robot_full.urdf.xacro (robot description, xacro)
@@ -1,9 +1 @@
-<?xml version="1.0"?>
-<robot xmlns:xacro="http://www.ros.org/wiki/xacro" name="jaguar_robot_full">
-    <xacro:arg name="initial_positions_file" default="initial_positions.yaml" />
-    <!-- Import jaguar_robot_full urdf file -->
-    <xacro:include filename="$(find jaguar_robot_full_description)/urdf/jaguar_robot_full.xacro" />
-    <!-- Import control_xacro -->
-    <xacro:include filename="jaguar_robot_full.ros2_control.xacro" />
-    <xacro:jaguar_robot_full_ros2_control name="FakeSystem" initial_positions_file="$(arg initial_positions_file)"/>
-</robot>
+/home/arepo/TMR2026_Rescue/jaguar/arm/src/jaguar_full/config/jaguar_robot_full.urdf.xacro
